File: pi2micro4.kicad_pcb (KiCad board)
At the start: 2 copper layers, 57.8 x 69.8 mm, 31 parts, among them K1 CONN_3, K2 CONN_3, M1 microduino_base, M2 microduino_base, M3 microduino_base, M4 microduino_base, P1 CONN_13X2, SW1 RST, U1 NCP1117ST33T3G, U2 txs0104e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

Commit message: 6 conectores para servos
Parts:
- added K3: CONN_S7, SIL-3, F.Cu at (143.5, 147.3)
- added K4: CONN_S10, SIL-3, F.Cu at (135.9, 147.3)
- added K5: CONN_S8, SIL-3, F.Cu at (141.0, 147.3)
- added K6: CONN_S11, SIL-3, F.Cu at (133.3, 147.3)
- added K7: CONN_S9, SIL-3, F.Cu at (138.4, 147.3)
- added K8: CONN_S12, SIL-3, F.Cu at (130.8, 147.3)
- moved K2 18.5 mm to (114.3, 144.8)
- moved K1 17.9 mm to (123.8, 144.8)
- moved U3 8.79 mm to (134.7, 114.5)
- moved R1 6.43 mm to (108.0, 144.5), turned to 270 degrees
- moved D1 5.06 mm to (106.2, 144.5), turned to 90 degrees
- moved R2 3.82 mm to (103.6, 144.5), turned to 270 degrees
- moved D2 2.50 mm to (101.9, 144.5), turned to 90 degrees
- moved C6 1.73 mm to (147.3, 95.7)
- moved C5 1.15 mm to (139.7, 100.8)
- moved C3 0.99 mm to (146.9, 87.4)
- moved C4 0.74 mm to (146.5, 83.5), turned to 0 degrees
Routing:
- net GND: track 451.3 -> 270.8 mm, vias 19 -> 1
- net /3V3_RB: track 98.7 -> 185.1 mm
- net /D6: track 162.4 -> 120.8 mm, vias 0 -> 1
- net /D4: track 135.9 -> 97.6 mm, vias 0 -> 1
- net /RST: track 188.2 -> 216.0 mm
- net +5V: track 260.9 -> 236.5 mm
- net Net-(K1-Pad2): track 43.4 -> 66.7 mm, vias 2 -> 0
- net /D7: track 136.1 -> 157.6 mm
- net /A1: track 86.7 -> 66.6 mm
- net /D5: track 131.9 -> 112.6 mm, vias 0 -> 1
- net /D2: track 96.4 -> 78.4 mm
- net Net-(K2-Pad2): track 103.2 -> 87.0 mm, vias 1 -> 0
- net /A4: track 89.5 -> 77.4 mm, vias 1 -> 2
- net /A2: track 68.9 -> 57.1 mm, vias 0 -> 2
- net /D8: track 128.6 -> 117.7 mm, vias 0 -> 1
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Other:
- board text added: "D10"
- board text added: "D11"
- board text added: "D12"
- board text added: "D7"
- board text added: "D8"
- board text added: "D9"
